File: Kicad/bmc.sch (KiCad schematic (older format))
At the start: 27 parts, among them J1101 Header, J1102 Header, J1103 Conn_01x05, J1104 Double-mini-DIN-6, SW1101 SW_DIP_x01, SW1102 SW_DIP_x01, U1101 STM32F031K6T6

Commit message: Switching some parts over to the CPL.
Parts:
- C1101, C1102: Digikey BC1150CT-ND -> (none); MPN K104K15X7RF5TL2 -> CPL-CAP-X7R-0805-100NF-50V; Manufacturer Vishay -> CPL; Mouser 594-K104K15X7RF5TL2 -> (none)
- C1103: value 4u7 10V -> 4u7 16V; Digikey 1276-6464-1-ND -> (none); MPN CL21A475KPFNNNG -> CPL-CAP-X5R-0805-4.7UF-25V; Manufacturer Samsung -> CPL
- C1105: value 1u 10V -> 1u 16V; Digikey 1276-6471-1-ND -> (none); MPN CL21B105KOFNNNG -> CPL-CAP-X7R-0805-1UF-25V; Manufacturer Samsung -> CPL
- D1101, D1102: MPN 151031SS06000 -> CPL-LED-3MM-RED; Manufacturer Würth -> CPL
- R1101, R1102, R1103, R1104: Digikey RMCF0805FT1K00-ND -> (none); MPN RMCF0805FT1K00 -> CPL-RES-0805-1K-0.125W; Manufacturer Stackpole -> CPL
- R1105, R1106, R1107, R1108, R1109, R1110, R1111: Digikey RMCF0805FT10K0-ND -> (none); MPN RMCF0805FT10K0 -> CPL-RES-0805-10K-0.125W; Manufacturer Stackpole -> CPL
Changed lines of the file:
@@
 P 5550 5000
 F 0 "C1103" H 5650 5050 50  0000 L CNN
-F 1 "4u7 10V" H 5650 4950 50  0000 L CNN
+F 1 "4u7 16V" H 5650 4950 50  0000 L CNN
 F 2 "Capacitor_SMD:C_0805_2012Metric_Pad1.18x1.45mm_HandSolder" H 5588 4850 50  0001 C CNN
 F 3 "~" H 5550 5000 50  0001 C CNN
 F 4 "0" H 5550 5000 50  0001 C CNN "DNP"
-F 5 "1276-6464-1-ND" H 5550 5000 50  0001 C CNN "Digikey"
-F 6 "CL21A475KPFNNNG" H 5550 5000 50  0001 C CNN "MPN"
-F 7 "Samsung" H 5550 5000 50  0001 C CNN "Manufacturer"
+F 5 "" H 5550 5000 50  0001 C CNN "Digikey"
+F 6 "CPL-CAP-X5R-0805-4.7UF-25V" H 5550 5000 50  0001 C CNN "MPN"
+F 7 "CPL" H 5550 5000 50  0001 C CNN "Manufacturer"
 	1    5550 5000
 	1    0    0    -1
@@
 F 6 "~" H 3425 3725 50  0001 C CNN "MPN"
 F 7 "~" H 3425 3725 50  0001 C CNN "Manufacturer"
-F 8 "" H 3425 3725 50  0001 C CNN "Mouser"
+F 8 "~" H 3425 3725 50  0001 C CNN "Mouser"
 	1    3425 3725
 	1    0    0    -1
@@
 F 6 "~" H 3425 2975 50  0001 C CNN "MPN"
 F 7 "~" H 3425 2975 50  0001 C CNN "Manufacturer"
-F 8 "" H 3425 2975 50  0001 C CNN "Mouser"
+F 8 "~" H 3425 2975 50  0001 C CNN "Mouser"
 	1    3425 2975
 	1    0    0    -1
@@
 F 3 "~" H 5100 5000 50  0001 C CNN
 F 4 "0" H 5100 5000 50  0001 C CNN "DNP"
-F 5 "BC1150CT-ND" H 5100 5000 50  0001 C CNN "Digikey"
-F 6 "K104K15X7RF5TL2" H 5100 5000 50  0001 C CNN "MPN"
-F 7 "Vishay" H 5100 5000 50  0001 C CNN "Manufacturer"
-F 8 "594-K104K15X7RF5TL2" H 5100 5000 50  0001 C CNN "Mouser"
+F 5 "" H 5100 5000 50  0001 C CNN "Digikey"
+F 6 "CPL-CAP-X7R-0805-100NF-50V" H 5100 5000 50  0001 C CNN "MPN"
+F 7 "CPL" H 5100 5000 50  0001 C CNN "Manufacturer"
+F 8 "" H 5100 5000 50  0001 C CNN "Mouser"
 	1    5100 5000
 	1    0    0    -1
@@
 F 3 "~" H 4650 5000 50  0001 C CNN
 F 4 "0" H 4650 5000 50  0001 C CNN "DNP"
-F 5 "BC1150CT-ND" H 4650 5000 50  0001 C CNN "Digikey"
-F 6 "K104K15X7RF5TL2" H 4650 5000 50  0001 C CNN "MPN"
-F 7 "Vishay" H 4650 5000 50  0001 C CNN "Manufacturer"
-F 8 "594-K104K15X7RF5TL2" H 4650 5000 50  0001 C CNN "Mouser"
+F 5 "" H 4650 5000 50  0001 C CNN "Digikey"
+F 6 "CPL-CAP-X7R-0805-100NF-50V" H 4650 5000 50  0001 C CNN "MPN"
+F 7 "CPL" H 4650 5000 50  0001 C CNN "Manufacturer"
+F 8 "" H 4650 5000 50  0001 C CNN "Mouser"
 	1    4650 5000
 	1    0    0    -1
@@
 F 3 "~" H 4100 2125 50  0001 C CNN
 F 4 "0" H 4100 2125 50  0001 C CNN "DNP"
-F 5 "RMCF0805FT10K0-ND" H 4100 2125 50  0001 C CNN "Digikey"
-F 6 "RMCF0805FT10K0" H 4100 2125 50  0001 C CNN "MPN"
-F 7 "Stackpole" H 4100 2125 50  0001 C CNN "Manufacturer"
+F 5 "" H 4100 2125 50  0001 C CNN "Digikey"
+F 6 "CPL-RES-0805-10K-0.125W" H 4100 2125 50  0001 C CNN "MPN"
+F 7 "CPL" H 4100 2125 50  0001 C CNN "Manufacturer"
 	1    4100 2125
 	1    0    0    -1
@@
 F 3 "~" H 2850 5250 50  0001 C CNN
 F 4 "0" H 2850 5250 50  0001 C CNN "DNP"
-F 5 "RMCF0805FT1K00-ND" H 2850 5250 50  0001 C CNN "Digikey"
-F 6 "RMCF0805FT1K00" H 2850 5250 50  0001 C CNN "MPN"
-F 7 "Stackpole" H 2850 5250 50  0001 C CNN "Manufacturer"
+F 5 "" H 2850 5250 50  0001 C CNN "Digikey"
+F 6 "CPL-RES-0805-1K-0.125W" H 2850 5250 50  0001 C CNN "MPN"
+F 7 "CPL" H 2850 5250 50  0001 C CNN "Manufacturer"
 	1    2850 5250
 	1    0    0    -1
@@
 F 3 "~" H 3050 5250 50  0001 C CNN
 F 4 "0" H 3050 5250 50  0001 C CNN "DNP"
-F 5 "RMCF0805FT1K00-ND" H 3050 5250 50  0001 C CNN "Digikey"
-F 6 "RMCF0805FT1K00" H 3050 5250 50  0001 C CNN "MPN"
-F 7 "Stackpole" H 3050 5250 50  0001 C CNN "Manufacturer"
+F 5 "" H 3050 5250 50  0001 C CNN "Digikey"
+F 6 "CPL-RES-0805-1K-0.125W" H 3050 5250 50  0001 C CNN "MPN"
+F 7 "CPL" H 3050 5250 50  0001 C CNN "Manufacturer"
 	1    3050 5250
 	-1   0    0    -1
@@
 F 4 "0" H 3050 5650 50  0001 C CNN "DNP"
 F 5 "732-5006-ND" H 3050 5650 50  0001 C CNN "Digikey"
-F 6 "151031SS06000" H 3050 5650 50  0001 C CNN "MPN"
-F 7 "Würth" H 3050 5650 50  0001 C CNN "Manufacturer"
+F 6 "CPL-LED-3MM-RED" H 3050 5650 50  0001 C CNN "MPN"
+F 7 "CPL" H 3050 5650 50  0001 C CNN "Manufacturer"
 F 8 "151031SS06000" H 3050 5650 50  0001 C CNN "Mouser"
 	1    3050 5650
@@
 F 3 "~" H 1575 5250 50  0001 C CNN
 F 4 "0" H 1575 5250 50  0001 C CNN "DNP"
-F 5 "RMCF0805FT1K00-ND" H 1575 5250 50  0001 C CNN "Digikey"
-F 6 "RMCF0805FT1K00" H 1575 5250 50  0001 C CNN "MPN"
-F 7 "Stackpole" H 1575 5250 50  0001 C CNN "Manufacturer"
+F 5 "" H 1575 5250 50  0001 C CNN "Digikey"
+F 6 "CPL-RES-0805-1K-0.125W" H 1575 5250 50  0001 C CNN "MPN"
+F 7 "CPL" H 1575 5250 50  0001 C CNN "Manufacturer"
 	1    1575 5250
 	-1   0    0    -1
@@
 F 3 "~" H 1775 5250 50  0001 C CNN
 F 4 "0" H 1775 5250 50  0001 C CNN "DNP"
-F 5 "RMCF0805FT1K00-ND" H 1775 5250 50  0001 C CNN "Digikey"
-F 6 "RMCF0805FT1K00" H 1775 5250 50  0001 C CNN "MPN"
-F 7 "Stackpole" H 1775 5250 50  0001 C CNN "Manufacturer"
+F 5 "" H 1775 5250 50  0001 C CNN "Digikey"
+F 6 "CPL-RES-0805-1K-0.125W" H 1775 5250 50  0001 C CNN "MPN"
+F 7 "CPL" H 1775 5250 50  0001 C CNN "Manufacturer"
 	1    1775 5250
 	-1   0    0    -1
@@
 F 4 "0" H 1775 5650 50  0001 C CNN "DNP"
 F 5 "732-5006-ND" H 1775 5650 50  0001 C CNN "Digikey"
-F 6 "151031SS06000" H 1775 5650 50  0001 C CNN "MPN"
-F 7 "Würth" H 1775 5650 50  0001 C CNN "Manufacturer"
+F 6 "CPL-LED-3MM-RED" H 1775 5650 50  0001 C CNN "MPN"
+F 7 "CPL" H 1775 5650 50  0001 C CNN "Manufacturer"
 F 8 "151031SS06000" H 1775 5650 50  0001 C CNN "Mouser"
 	1    1775 5650
@@
 P 6550 5000
 F 0 "C1105" H 6650 5050 50  0000 L CNN
-F 1 "1u 10V" H 6650 4950 50  0000 L CNN
+F 1 "1u 16V" H 6650 4950 50  0000 L CNN
 F 2 "Capacitor_SMD:C_0805_2012Metric_Pad1.18x1.45mm_HandSolder" H 6588 4850 50  0001 C CNN
 F 3 "~" H 6550 5000 50  0001 C CNN
 F 4 "0" H 6550 5000 50  0001 C CNN "DNP"
-F 5 "1276-6471-1-ND" H 6550 5000 50  0001 C CNN "Digikey"
-F 6 "CL21B105KOFNNNG" H 6550 5000 50  0001 C CNN "MPN"
-F 7 "Samsung" H 6550 5000 50  0001 C CNN "Manufacturer"
+F 5 "" H 6550 5000 50  0001 C CNN "Digikey"
+F 6 "CPL-CAP-X7R-0805-1UF-25V" H 6550 5000 50  0001 C CNN "MPN"
+F 7 "CPL" H 6550 5000 50  0001 C CNN "Manufacturer"
 	1    6550 5000
 	1    0    0    -1
@@
 F 3 "~" H 8925 2975 50  0001 C CNN
 F 4 "0" H 8925 2975 50  0001 C CNN "DNP"
-F 5 "RMCF0805FT10K0-ND" H 8925 2975 50  0001 C CNN "Digikey"
-F 6 "RMCF0805FT10K0" H 8925 2975 50  0001 C CNN "MPN"
-F 7 "Stackpole" H 8925 2975 50  0001 C CNN "Manufacturer"
+F 5 "" H 8925 2975 50  0001 C CNN "Digikey"
+F 6 "CPL-RES-0805-10K-0.125W" H 8925 2975 50  0001 C CNN "MPN"
+F 7 "CPL" H 8925 2975 50  0001 C CNN "Manufacturer"
 	1    8925 2975
 	1    0    0    -1
@@
 F 3 "~" H 8925 2575 50  0001 C CNN
 F 4 "0" H 8925 2575 50  0001 C CNN "DNP"
-F 5 "RMCF0805FT10K0-ND" H 8925 2575 50  0001 C CNN "Digikey"
-F 6 "RMCF0805FT10K0" H 8925 2575 50  0001 C CNN "MPN"
-F 7 "Stackpole" H 8925 2575 50  0001 C CNN "Manufacturer"
+F 5 "" H 8925 2575 50  0001 C CNN "Digikey"
+F 6 "CPL-RES-0805-10K-0.125W" H 8925 2575 50  0001 C CNN "MPN"
+F 7 "CPL" H 8925 2575 50  0001 C CNN "Manufacturer"
 	1    8925 2575
 	1    0    0    -1
@@
 F 3 "~" H 8925 2225 50  0001 C CNN
 F 4 "0" H 8925 2225 50  0001 C CNN "DNP"
-F 5 "RMCF0805FT10K0-ND" H 8925 2225 50  0001 C CNN "Digikey"
-F 6 "RMCF0805FT10K0" H 8925 2225 50  0001 C CNN "MPN"
-F 7 "Stackpole" H 8925 2225 50  0001 C CNN "Manufacturer"
+F 5 "" H 8925 2225 50  0001 C CNN "Digikey"
+F 6 "CPL-RES-0805-10K-0.125W" H 8925 2225 50  0001 C CNN "MPN"
+F 7 "CPL" H 8925 2225 50  0001 C CNN "Manufacturer"
 	1    8925 2225
 	1    0    0    -1
@@
 F 3 "~" H 8475 2175 50  0001 C CNN
 F 4 "0" H 8475 2175 50  0001 C CNN "DNP"
-F 5 "RMCF0805FT10K0-ND" H 8475 2175 50  0001 C CNN "Digikey"
-F 6 "RMCF0805FT10K0" H 8475 2175 50  0001 C CNN "MPN"
-F 7 "Stackpole" H 8475 2175 50  0001 C CNN "Manufacturer"
+F 5 "" H 8475 2175 50  0001 C CNN "Digikey"
+F 6 "CPL-RES-0805-10K-0.125W" H 8475 2175 50  0001 C CNN "MPN"
+F 7 "CPL" H 8475 2175 50  0001 C CNN "Manufacturer"
 	1    8475 2175
 	1    0    0    -1
@@
 F 3 "~" H 8475 1775 50  0001 C CNN
 F 4 "0" H 8475 1775 50  0001 C CNN "DNP"
-F 5 "RMCF0805FT10K0-ND" H 8475 1775 50  0001 C CNN "Digikey"
-F 6 "RMCF0805FT10K0" H 8475 1775 50  0001 C CNN "MPN"
-F 7 "Stackpole" H 8475 1775 50  0001 C CNN "Manufacturer"
+F 5 "" H 8475 1775 50  0001 C CNN "Digikey"
+F 6 "CPL-RES-0805-10K-0.125W" H 8475 1775 50  0001 C CNN "MPN"
+F 7 "CPL" H 8475 1775 50  0001 C CNN "Manufacturer"
 	1    8475 1775
 	1    0    0    -1
@@
 F 3 "~" H 8000 3950 50  0001 C CNN
 F 4 "0" H 8000 3950 50  0001 C CNN "DNP"
-F 5 "RMCF0805FT10K0-ND" H 8000 3950 50  0001 C CNN "Digikey"
-F 6 "RMCF0805FT10K0" H 8000 3950 50  0001 C CNN "MPN"
-F 7 "Stackpole" H 8000 3950 50  0001 C CNN "Manufacturer"
+F 5 "" H 8000 3950 50  0001 C CNN "Digikey"
+F 6 "CPL-RES-0805-10K-0.125W" H 8000 3950 50  0001 C CNN "MPN"
+F 7 "CPL" H 8000 3950 50  0001 C CNN "Manufacturer"
 	1    8000 3950
 	-1   0    0    -1

Commit message: Fixing some review comments.
* PCB has rounded corners.
* Add JLCPCB part numbers for SMT parts
* Fixed Fab layer
* Renumbered Slots
* Mounting holes do not have thermal relief

Closes #13 #12 and #10
Parts:
- C1101, C1102: LCSC Part# (none) -> C49678
- C1103: LCSC Part# (none) -> C1779
- C1104: LCSC Part# (none) -> C1710
- C1105: LCSC Part# (none) -> C28323
- R1101, R1102, R1103, R1104: LCSC Part# (none) -> C17513
- R1105, R1106, R1107, R1108, R1109, R1110, R1111: LCSC Part# (none) -> C17414
- U1101: LCSC Part# (none) -> C526904
Changed lines of the file:
@@
 F 6 "CPL-CAP-X5R-0805-4.7UF-25V" H 5550 5000 50  0001 C CNN "MPN"
 F 7 "CPL" H 5550 5000 50  0001 C CNN "Manufacturer"
+F 8 "C1779" H 5550 5000 50  0001 C CNN "LCSC Part#"
 	1    5550 5000
 	1    0    0    -1
@@
 F 7 "~" H 3425 3725 50  0001 C CNN "Manufacturer"
 F 8 "~" H 3425 3725 50  0001 C CNN "Mouser"
+F 9 "~" H 3425 3725 50  0001 C CNN "LCSC Part#"
 	1    3425 3725
 	1    0    0    -1
@@
 F 7 "~" H 3425 2975 50  0001 C CNN "Manufacturer"
 F 8 "~" H 3425 2975 50  0001 C CNN "Mouser"
+F 9 "~" H 3425 2975 50  0001 C CNN "LCSC Part#"
 	1    3425 2975
 	1    0    0    -1
@@
 F 7 "Kycon" H 9075 5725 50  0001 C CNN "Manufacturer"
 F 8 "806-KMDGX-6S/6S-S4N" H 9075 5725 50  0001 C CNN "Mouser"
+F 9 "~" H 9075 5725 50  0001 C CNN "LCSC Part#"
 	1    9075 5725
 	1    0    0    -1
@@
 F 7 "CPL" H 5100 5000 50  0001 C CNN "Manufacturer"
 F 8 "" H 5100 5000 50  0001 C CNN "Mouser"
+F 9 "C49678" H 5100 5000 50  0001 C CNN "LCSC Part#"
 	1    5100 5000
 	1    0    0    -1
@@
 F 7 "0" H 6225 2375 50  0001 C CNN "DNP"
 F 8 "511-STM32F031K6T6" H 6225 2375 50  0001 C CNN "Mouser"
+F 9 "C526904" H 6225 2375 50  0001 C CNN "LCSC Part#"
 	1    6225 2375
 	1    0    0    -1
@@
 F 6 "~" H 3800 1875 50  0001 C CNN "MPN"
 F 7 "~" H 3800 1875 50  0001 C CNN "Manufacturer"
+F 8 "~" H 3800 1875 50  0001 C CNN "LCSC Part#"
 	1    3800 1875
 	1    0    0    -1
@@
 F 7 "CPL" H 4650 5000 50  0001 C CNN "Manufacturer"
 F 8 "" H 4650 5000 50  0001 C CNN "Mouser"
+F 9 "C49678" H 4650 5000 50  0001 C CNN "LCSC Part#"
 	1    4650 5000
 	1    0    0    -1
@@
 F 6 "~" H 4225 1350 50  0001 C CNN "MPN"
 F 7 "~" H 4225 1350 50  0001 C CNN "Manufacturer"
+F 8 "~" H 4225 1350 50  0001 C CNN "LCSC Part#"
 	1    4225 1350
 	-1   0    0    1
@@
 F 6 "CPL-RES-0805-10K-0.125W" H 4100 2125 50  0001 C CNN "MPN"
 F 7 "CPL" H 4100 2125 50  0001 C CNN "Manufacturer"
+F 8 "C17414" H 4100 2125 50  0001 C CNN "LCSC Part#"
 	1    4100 2125
 	1    0    0    -1
@@
 F 6 "CPL-RES-0805-1K-0.125W" H 2850 5250 50  0001 C CNN "MPN"
 F 7 "CPL" H 2850 5250 50  0001 C CNN "Manufacturer"
+F 8 "C17513" H 2850 5250 50  0001 C CNN "LCSC Part#"
 	1    2850 5250
 	1    0    0    -1
@@
 F 6 "CPL-RES-0805-1K-0.125W" H 3050 5250 50  0001 C CNN "MPN"
 F 7 "CPL" H 3050 5250 50  0001 C CNN "Manufacturer"
+F 8 "C17513" H 3050 5250 50  0001 C CNN "LCSC Part#"
 	1    3050 5250
 	-1   0    0    -1
@@
 F 7 "CPL" H 3050 5650 50  0001 C CNN "Manufacturer"
 F 8 "151031SS06000" H 3050 5650 50  0001 C CNN "Mouser"
+F 9 "~" H 3050 5650 50  0001 C CNN "LCSC Part#"
 	1    3050 5650
 	0    -1   -1   0
@@
 F 6 "~" H 2650 5600 50  0001 C CNN "MPN"
 F 7 "~" H 2650 5600 50  0001 C CNN "Manufacturer"
+F 8 "~" H 2650 5600 50  0001 C CNN "LCSC Part#"
 	1    2650 5600
 	1    0    0    -1
@@
 F 6 "CPL-RES-0805-1K-0.125W" H 1575 5250 50  0001 C CNN "MPN"
 F 7 "CPL" H 1575 5250 50  0001 C CNN "Manufacturer"
+F 8 "C17513" H 1575 5250 50  0001 C CNN "LCSC Part#"
 	1    1575 5250
 	-1   0    0    -1
@@
 F 6 "CPL-RES-0805-1K-0.125W" H 1775 5250 50  0001 C CNN "MPN"
 F 7 "CPL" H 1775 5250 50  0001 C CNN "Manufacturer"
+F 8 "C17513" H 1775 5250 50  0001 C CNN "LCSC Part#"
 	1    1775 5250
 	-1   0    0    -1
@@
 F 7 "CPL" H 1775 5650 50  0001 C CNN "Manufacturer"
 F 8 "151031SS06000" H 1775 5650 50  0001 C CNN "Mouser"
+F 9 "~" H 1775 5650 50  0001 C CNN "LCSC Part#"
 	1    1775 5650
 	0    -1   -1   0
@@
 F 6 "~" H 1375 5600 50  0001 C CNN "MPN"
 F 7 "~" H 1375 5600 50  0001 C CNN "Manufacturer"
+F 8 "~" H 1375 5600 50  0001 C CNN "LCSC Part#"
 	1    1375 5600
 	1    0    0    -1
@@
 F 7 "Bourns" H 10125 5100 50  0001 C CNN "Manufacturer"
 F 8 "652-4605X-1LF-2.7K" H 10125 5100 50  0001 C CNN "Mouser"
+F 9 "~" H 10125 5100 50  0001 C CNN "LCSC Part#"
 	1    10125 5100
 	1    0    0    -1
@@
 F 6 "CPL-CAP-X7R-0805-1UF-25V" H 6550 5000 50  0001 C CNN "MPN"
 F 7 "CPL" H 6550 5000 50  0001 C CNN "Manufacturer"
+F 8 "C28323" H 6550 5000 50  0001 C CNN "LCSC Part#"
 	1    6550 5000
 	1    0    0    -1
@@
 F 6 "CL21B103KCANNNC" H 6100 5000 50  0001 C CNN "MPN"
 F 7 "Samsung" H 6100 5000 50  0001 C CNN "Manufacturer"
+F 8 "C1710" H 6100 5000 50  0001 C CNN "LCSC Part#"
 	1    6100 5000
 	1    0    0    -1
@@
 F 6 "CPL-RES-0805-10K-0.125W" H 8925 2975 50  0001 C CNN "MPN"
 F 7 "CPL" H 8925 2975 50  0001 C CNN "Manufacturer"
+F 8 "C17414" H 8925 2975 50  0001 C CNN "LCSC Part#"
 	1    8925 2975
 	1    0    0    -1
@@
 F 6 "CPL-RES-0805-10K-0.125W" H 8925 2575 50  0001 C CNN "MPN"
 F 7 "CPL" H 8925 2575 50  0001 C CNN "Manufacturer"
+F 8 "C17414" H 8925 2575 50  0001 C CNN "LCSC Part#"
 	1    8925 2575
 	1    0    0    -1
@@
 F 6 "CPL-RES-0805-10K-0.125W" H 8925 2225 50  0001 C CNN "MPN"
 F 7 "CPL" H 8925 2225 50  0001 C CNN "Manufacturer"
+F 8 "C17414" H 8925 2225 50  0001 C CNN "LCSC Part#"
 	1    8925 2225
 	1    0    0    -1
@@
 F 6 "CPL-RES-0805-10K-0.125W" H 8475 2175 50  0001 C CNN "MPN"
 F 7 "CPL" H 8475 2175 50  0001 C CNN "Manufacturer"
+F 8 "C17414" H 8475 2175 50  0001 C CNN "LCSC Part#"
 	1    8475 2175
 	1    0    0    -1
@@
 F 6 "CPL-RES-0805-10K-0.125W" H 8475 1775 50  0001 C CNN "MPN"
 F 7 "CPL" H 8475 1775 50  0001 C CNN "Manufacturer"
+F 8 "C17414" H 8475 1775 50  0001 C CNN "LCSC Part#"
 	1    8475 1775
 	1    0    0    -1
@@
 F 6 "CPL-RES-0805-10K-0.125W" H 8000 3950 50  0001 C CNN "MPN"
 F 7 "CPL" H 8000 3950 50  0001 C CNN "Manufacturer"
+F 8 "C17414" H 8000 3950 50  0001 C CNN "LCSC Part#"
 	1    8000 3950
 	-1   0    0    -1
