File: Kicad/bmc.sch (KiCad schematic (older format))
At the start: 32 parts, among them J1001 Header, J1002 Header, J1003 Conn_01x05, J1004 Double-mini-DIN-6, SW1001 SW_DIP_x01, SW1002 SW_DIP_x01, SW1003 SW_DIP_x01, SW1004 SW_DIP_x01, U1001 STM32F031K6T6

Commit message: Renamed LED/button headers to be consistent.
Parts:
- J1003: renamed from SW1002; value SW_DIP_x01 -> CONN 1x02
- J1004: renamed from SW1003; value SW_DIP_x01 -> CONN 1x02
- SW1001: value SW_DIP_x01 -> SPST 6mm
- SW1002: renamed from SW1004; value SW_DIP_x01 -> SPST 6mm
- renumbered JP1001 to J1005, J1003 to J1006, J1004 to J1007
Other:
- moved on the sheet: J1004, SW1002
