File: Kicad/io_exp.sch (KiCad schematic (older format))
At the start: 4 parts, among them U1001 MCP23S17_SO, U1002 74HC245

Commit message: Added expansion header.
Involved rerouting quite a few things.
Also added through-hole switches for power/reset.
Parts:
- renumbered C1001 to C901, C1002 to C902, U1001 to U901, U1002 to U902
Changed lines of the file:
@@
 $EndDescr
 $Comp
-L neotron-pico:MCP23S17_SO U1001
+L neotron-pico:MCP23S17_SO U901
 U 1 1 60EED5B0
 P 4425 3050
-F 0 "U1001" H 3975 4025 50  0000 C CNN
+F 0 "U901" H 3975 4025 50  0000 C CNN
 F 1 "MCP23S17_SO" H 4775 4025 50  0000 C CNN
 F 2 "Package_SO:SOIC-28W_7.5x17.9mm_P1.27mm" H 4625 2050 50  0001 L CNN
@@
 	5500 2100 5625 2100
 $Comp
-L 74xx:74HC245 U1002
+L 74xx:74HC245 U902
 U 1 1 60F0F5AC
 P 6050 3650
-F 0 "U1002" H 5800 4325 50  0000 C CNN
+F 0 "U902" H 5800 4325 50  0000 C CNN
 F 1 "74HC245" H 6275 4325 50  0000 C CNN
 F 2 "Package_SO:SO-20_12.8x7.5mm_P1.27mm" H 6050 3650 50  0001 C CNN
@@
 	5425 4150 5550 4150
 $Comp
-L power:GND #PWR01005
+L power:GND #PWR0905
 U 1 1 60F11A9D
 P 6050 4550
-F 0 "#PWR01005" H 6050 4300 50  0001 C CNN
+F 0 "#PWR0905" H 6050 4300 50  0001 C CNN
 F 1 "GND" H 6055 4377 50  0000 C CNN
 F 2 "" H 6050 4550 50  0001 C CNN
@@
 	6050 4550 6050 4450
 $Comp
-L power:GND #PWR01003
+L power:GND #PWR0903
 U 1 1 60F121EF
 P 5500 4550
-F 0 "#PWR01003" H 5500 4300 50  0001 C CNN
+F 0 "#PWR0903" H 5500 4300 50  0001 C CNN
 F 1 "GND" H 5505 4377 50  0000 C CNN
 F 2 "" H 5500 4550 50  0001 C CNN
@@
 	5125 3850 5550 3850
 $Comp
-L power:+3.3V #PWR01001
+L power:+3.3V #PWR0901
 U 1 1 60F1A105
 P 4425 1875
-F 0 "#PWR01001" H 4425 1725 50  0001 C CNN
+F 0 "#PWR0901" H 4425 1725 50  0001 C CNN
 F 1 "+3.3V" H 4440 2048 50  0000 C CNN
 F 2 "" H 4425 1875 50  0001 C CNN
@@
 	4425 1875 4425 1950
 $Comp
-L power:+3.3V #PWR01004
+L power:+3.3V #PWR0904
 U 1 1 60F1ADA6
 P 6050 2775
-F 0 "#PWR01004" H 6050 2625 50  0001 C CNN
+F 0 "#PWR0904" H 6050 2625 50  0001 C CNN
 F 1 "+3.3V" H 6065 2948 50  0000 C CNN
 F 2 "" H 6050 2775 50  0001 C CNN
@@
 	6050 2775 6050 2850
 $Comp
-L power:GND #PWR01002
+L power:GND #PWR0902
 U 1 1 60F1C2DF
 P 4425 4550
-F 0 "#PWR01002" H 4425 4300 50  0001 C CNN
+F 0 "#PWR0902" H 4425 4300 50  0001 C CNN
 F 1 "GND" H 4430 4377 50  0000 C CNN
 F 2 "" H 4425 4550 50  0001 C CNN
@@
 	3550 3850 3550 4225
 $Comp
-L power:+3.3V #PWR01006
+L power:+3.3V #PWR0906
 U 1 1 60F1F612
 P 7900 2250
-F 0 "#PWR01006" H 7900 2100 50  0001 C CNN
+F 0 "#PWR0906" H 7900 2100 50  0001 C CNN
 F 1 "+3.3V" H 7915 2423 50  0000 C CNN
 F 2 "" H 7900 2250 50  0001 C CNN
@@
 $EndComp
 $Comp
-L power:GND #PWR01007
+L power:GND #PWR0907
 U 1 1 60F1F772
 P 7900 2750
-F 0 "#PWR01007" H 7900 2500 50  0001 C CNN
+F 0 "#PWR0907" H 7900 2500 50  0001 C CNN
 F 1 "GND" H 7905 2577 50  0000 C CNN
 F 2 "" H 7900 2750 50  0001 C CNN
@@
 P 7900 2500
 AR Path="/5FEF6B08/60F34F63" Ref="C?"  Part="1"
-AR Path="/6069D32A/60F34F63" Ref="C1001"  Part="1"
-F 0 "C1001" H 8015 2546 50  0000 L CNN
+AR Path="/6069D32A/60F34F63" Ref="C901"  Part="1"
+F 0 "C901" H 8015 2546 50  0000 L CNN
 F 1 "100nF" H 8015 2455 50  0000 L CNN
 F 2 "Capacitor_SMD:C_0805_2012Metric_Pad1.18x1.45mm_HandSolder" H 7938 2350 50  0001 C CNN
@@
 P 8375 2500
 AR Path="/5FEF6B08/60F36BE4" Ref="C?"  Part="1"
-AR Path="/6069D32A/60F36BE4" Ref="C1002"  Part="1"
-F 0 "C1002" H 8490 2546 50  0000 L CNN
+AR Path="/6069D32A/60F36BE4" Ref="C902"  Part="1"
+F 0 "C902" H 8490 2546 50  0000 L CNN
 F 1 "100nF" H 8490 2455 50  0000 L CNN
 F 2 "Capacitor_SMD:C_0805_2012Metric_Pad1.18x1.45mm_HandSolder" H 8413 2350 50  0001 C CNN
