File: Kicad/dac4.sch (KiCad schematic (older format))
At the start: 10 parts

Commit message: Added expansion header.
Involved rerouting quite a few things.
Also added through-hole switches for power/reset.
Parts:
- renumbered R501 to R401, R502 to R402, R503 to R403, R504 to R404, R505 to R405, R506 to R406, R507 to R407, R508 to R408, R509 to R409, R510 to R410
Changed lines of the file:
@@
 $Descr A4 11693 8268
 encoding utf-8
-Sheet 5 11
+Sheet 4 11
 Title "Neotron Common Hardware - 4-bit DAC"
 Date "2021-06-10"
@@
 AR Path="/60677AF0/6068202E/60681FF9" Ref="R?"  Part="1"
 AR Path="/60677AF0/600A04B7/60681FF9" Ref="R?"  Part="1"
-AR Path="/60687F8A/5FEFB226/60681FF9" Ref="R503"  Part="1"
-AR Path="/60687F8A/6068202E/60681FF9" Ref="R603"  Part="1"
-AR Path="/60687F8A/600A04B7/60681FF9" Ref="R703"  Part="1"
-F 0 "R503" V 4100 3000 50  0000 C CNN
+AR Path="/60687F8A/5FEFB226/60681FF9" Ref="R403"  Part="1"
+AR Path="/60687F8A/6068202E/60681FF9" Ref="R503"  Part="1"
+AR Path="/60687F8A/600A04B7/60681FF9" Ref="R603"  Part="1"
+F 0 "R603" V 4100 3000 50  0000 C CNN
 F 1 "12k" V 4200 3000 50  0000 C CNN
 F 2 "Resistor_SMD:R_0805_2012Metric_Pad1.20x1.40mm_HandSolder" V 3930 3000 50  0001 C CNN
@@
 AR Path="/60677AF0/6068202E/60681FFB" Ref="R?"  Part="1"
 AR Path="/60677AF0/600A04B7/60681FFB" Ref="R?"  Part="1"
-AR Path="/60687F8A/5FEFB226/60681FFB" Ref="R505"  Part="1"
-AR Path="/60687F8A/6068202E/60681FFB" Ref="R605"  Part="1"
-AR Path="/60687F8A/600A04B7/60681FFB" Ref="R705"  Part="1"
-F 0 "R505" V 5100 3000 50  0000 C CNN
+AR Path="/60687F8A/5FEFB226/60681FFB" Ref="R405"  Part="1"
+AR Path="/60687F8A/6068202E/60681FFB" Ref="R505"  Part="1"
+AR Path="/60687F8A/600A04B7/60681FFB" Ref="R605"  Part="1"
+F 0 "R605" V 5100 3000 50  0000 C CNN
 F 1 "12k" V 5200 3000 50  0000 C CNN
 F 2 "Resistor_SMD:R_0805_2012Metric_Pad1.20x1.40mm_HandSolder" V 4930 3000 50  0001 C CNN
@@
 AR Path="/60677AF0/6068202E/60681FFC" Ref="R?"  Part="1"
 AR Path="/60677AF0/600A04B7/60681FFC" Ref="R?"  Part="1"
-AR Path="/60687F8A/5FEFB226/60681FFC" Ref="R507"  Part="1"
-AR Path="/60687F8A/6068202E/60681FFC" Ref="R607"  Part="1"
-AR Path="/60687F8A/600A04B7/60681FFC" Ref="R707"  Part="1"
-F 0 "R507" V 6100 3000 50  0000 C CNN
+AR Path="/60687F8A/5FEFB226/60681FFC" Ref="R407"  Part="1"
+AR Path="/60687F8A/6068202E/60681FFC" Ref="R507"  Part="1"
+AR Path="/60687F8A/600A04B7/60681FFC" Ref="R607"  Part="1"
+F 0 "R607" V 6100 3000 50  0000 C CNN
 F 1 "12k" V 6200 3000 50  0000 C CNN
 F 2 "Resistor_SMD:R_0805_2012Metric_Pad1.20x1.40mm_HandSolder" V 5930 3000 50  0001 C CNN
@@
 AR Path="/60677AF0/6068202E/60682000" Ref="#PWR?"  Part="1"
 AR Path="/60677AF0/600A04B7/60682000" Ref="#PWR?"  Part="1"
-AR Path="/60687F8A/5FEFB226/60682000" Ref="#PWR0501"  Part="1"
-AR Path="/60687F8A/6068202E/60682000" Ref="#PWR0601"  Part="1"
-AR Path="/60687F8A/600A04B7/60682000" Ref="#PWR0701"  Part="1"
-F 0 "#PWR0701" H 3500 3350 50  0001 C CNN
+AR Path="/60687F8A/5FEFB226/60682000" Ref="#PWR0401"  Part="1"
+AR Path="/60687F8A/6068202E/60682000" Ref="#PWR0501"  Part="1"
+AR Path="/60687F8A/600A04B7/60682000" Ref="#PWR0601"  Part="1"
+F 0 "#PWR0601" H 3500 3350 50  0001 C CNN
 F 1 "GND" H 3505 3427 50  0000 C CNN
 F 2 "" H 3500 3600 50  0001 C CNN
@@
 AR Path="/60677AF0/6068202E/60682001" Ref="#PWR?"  Part="1"
 AR Path="/60677AF0/600A04B7/60682001" Ref="#PWR?"  Part="1"
-AR Path="/60687F8A/5FEFB226/60682001" Ref="#PWR0502"  Part="1"
-AR Path="/60687F8A/6068202E/60682001" Ref="#PWR0602"  Part="1"
-AR Path="/60687F8A/600A04B7/60682001" Ref="#PWR0702"  Part="1"
-F 0 "#PWR0702" H 7550 3350 50  0001 C CNN
+AR Path="/60687F8A/5FEFB226/60682001" Ref="#PWR0402"  Part="1"
+AR Path="/60687F8A/6068202E/60682001" Ref="#PWR0502"  Part="1"
+AR Path="/60687F8A/600A04B7/60682001" Ref="#PWR0602"  Part="1"
+F 0 "#PWR0602" H 7550 3350 50  0001 C CNN
 F 1 "GND" H 7555 3427 50  0000 C CNN
 F 2 "" H 7550 3600 50  0001 C CNN
@@
 AR Path="/60677AF0/6068202E/60682002" Ref="R?"  Part="1"
 AR Path="/60677AF0/600A04B7/60682002" Ref="R?"  Part="1"
-AR Path="/60687F8A/5FEFB226/60682002" Ref="R502"  Part="1"
-AR Path="/60687F8A/6068202E/60682002" Ref="R602"  Part="1"
-AR Path="/60687F8A/600A04B7/60682002" Ref="R702"  Part="1"
-F 0 "R502" H 3570 3346 50  0000 L CNN
+AR Path="/60687F8A/5FEFB226/60682002" Ref="R402"  Part="1"
+AR Path="/60687F8A/6068202E/60682002" Ref="R502"  Part="1"
+AR Path="/60687F8A/600A04B7/60682002" Ref="R602"  Part="1"
+F 0 "R602" H 3570 3346 50  0000 L CNN
 F 1 "24k" H 3570 3255 50  0000 L CNN
 F 2 "Resistor_SMD:R_0805_2012Metric_Pad1.20x1.40mm_HandSolder" V 3430 3300 50  0001 C CNN
@@
 AR Path="/60677AF0/6068202E/5F5FD329" Ref="R?"  Part="1"
 AR Path="/60677AF0/600A04B7/5F5FD329" Ref="R?"  Part="1"
-AR Path="/60687F8A/5FEFB226/5F5FD329" Ref="R508"  Part="1"
-AR Path="/60687F8A/6068202E/5F5FD329" Ref="R608"  Part="1"
-AR Path="/60687F8A/600A04B7/5F5FD329" Ref="R708"  Part="1"
-F 0 "R508" H 6570 2746 50  0000 L CNN
+AR Path="/60687F8A/5FEFB226/5F5FD329" Ref="R408"  Part="1"
+AR Path="/60687F8A/6068202E/5F5FD329" Ref="R508"  Part="1"
+AR Path="/60687F8A/600A04B7/5F5FD329" Ref="R608"  Part="1"
+F 0 "R608" H 6570 2746 50  0000 L CNN
 F 1 "24k" H 6570 2655 50  0000 L CNN
 F 2 "Resistor_SMD:R_0805_2012Metric_Pad1.20x1.40mm_HandSolder" V 6430 2700 50  0001 C CNN
@@
 AR Path="/60677AF0/6068202E/60682003" Ref="R?"  Part="1"
 AR Path="/60677AF0/600A04B7/60682003" Ref="R?"  Part="1"
-AR Path="/60687F8A/5FEFB226/60682003" Ref="R506"  Part="1"
-AR Path="/60687F8A/6068202E/60682003" Ref="R606"  Part="1"
-AR Path="/60687F8A/600A04B7/60682003" Ref="R706"  Part="1"
-F 0 "R506" H 5570 2746 50  0000 L CNN
+AR Path="/60687F8A/5FEFB226/60682003" Ref="R406"  Part="1"
+AR Path="/60687F8A/6068202E/60682003" Ref="R506"  Part="1"
+AR Path="/60687F8A/600A04B7/60682003" Ref="R606"  Part="1"
+F 0 "R606" H 5570 2746 50  0000 L CNN
 F 1 "24k" H 5570 2655 50  0000 L CNN
 F 2 "Resistor_SMD:R_0805_2012Metric_Pad1.20x1.40mm_HandSolder" V 5430 2700 50  0001 C CNN
@@
 AR Path="/60677AF0/6068202E/60681FFA" Ref="R?"  Part="1"
 AR Path="/60677AF0/600A04B7/60681FFA" Ref="R?"  Part="1"
-AR Path="/60687F8A/5FEFB226/60681FFA" Ref="R504"  Part="1"
-AR Path="/60687F8A/6068202E/60681FFA" Ref="R604"  Part="1"
-AR Path="/60687F8A/600A04B7/60681FFA" Ref="R704"  Part="1"
-F 0 "R504" H 4570 2746 50  0000 L CNN
+AR Path="/60687F8A/5FEFB226/60681FFA" Ref="R404"  Part="1"
+AR Path="/60687F8A/6068202E/60681FFA" Ref="R504"  Part="1"
+AR Path="/60687F8A/600A04B7/60681FFA" Ref="R604"  Part="1"
+F 0 "R604" H 4570 2746 50  0000 L CNN
 F 1 "24k" H 4570 2655 50  0000 L CNN
 F 2 "Resistor_SMD:R_0805_2012Metric_Pad1.20x1.40mm_HandSolder" V 4430 2700 50  0001 C CNN
@@
 AR Path="/60677AF0/6068202E/5F5F4D05" Ref="R?"  Part="1"
 AR Path="/60677AF0/600A04B7/5F5F4D05" Ref="R?"  Part="1"
-AR Path="/60687F8A/5FEFB226/5F5F4D05" Ref="R501"  Part="1"
-AR Path="/60687F8A/6068202E/5F5F4D05" Ref="R601"  Part="1"
-AR Path="/60687F8A/600A04B7/5F5F4D05" Ref="R701"  Part="1"
-F 0 "R501" H 3570 2746 50  0000 L CNN
+AR Path="/60687F8A/5FEFB226/5F5F4D05" Ref="R401"  Part="1"
+AR Path="/60687F8A/6068202E/5F5F4D05" Ref="R501"  Part="1"
+AR Path="/60687F8A/600A04B7/5F5F4D05" Ref="R601"  Part="1"
+F 0 "R601" H 3570 2746 50  0000 L CNN
 F 1 "24k" H 3570 2655 50  0000 L CNN
 F 2 "Resistor_SMD:R_0805_2012Metric_Pad1.20x1.40mm_HandSolder" V 3430 2700 50  0001 C CNN
@@
 AR Path="/60677AF0/6068202E/60681FFD" Ref="R?"  Part="1"
 AR Path="/60677AF0/600A04B7/60681FFD" Ref="R?"  Part="1"
-AR Path="/60687F8A/5FEFB226/60681FFD" Ref="R509"  Part="1"
-AR Path="/60687F8A/6068202E/60681FFD" Ref="R609"  Part="1"
-AR Path="/60687F8A/600A04B7/60681FFD" Ref="R709"  Part="1"
-F 0 "R509" V 7100 3000 50  0000 C CNN
+AR Path="/60687F8A/5FEFB226/60681FFD" Ref="R409"  Part="1"
+AR Path="/60687F8A/6068202E/60681FFD" Ref="R509"  Part="1"
+AR Path="/60687F8A/600A04B7/60681FFD" Ref="R609"  Part="1"
+F 0 "R609" V 7100 3000 50  0000 C CNN
 F 1 "12k" V 7200 3000 50  0000 C CNN
 F 2 "Resistor_SMD:R_0805_2012Metric_Pad1.20x1.40mm_HandSolder" V 6930 3000 50  0001 C CNN
@@
 AR Path="/60677AF0/6068202E/60681FFF" Ref="R?"  Part="1"
 AR Path="/60677AF0/600A04B7/60681FFF" Ref="R?"  Part="1"
-AR Path="/60687F8A/5FEFB226/60681FFF" Ref="R510"  Part="1"
-AR Path="/60687F8A/6068202E/60681FFF" Ref="R610"  Part="1"
-AR Path="/60687F8A/600A04B7/60681FFF" Ref="R710"  Part="1"
-F 0 "R510" H 7620 3346 50  0000 L CNN
+AR Path="/60687F8A/5FEFB226/60681FFF" Ref="R410"  Part="1"
+AR Path="/60687F8A/6068202E/60681FFF" Ref="R510"  Part="1"
+AR Path="/60687F8A/600A04B7/60681FFF" Ref="R610"  Part="1"
+F 0 "R610" H 7620 3346 50  0000 L CNN
 F 1 "5490" H 7620 3255 50  0000 L CNN
 F 2 "Resistor_SMD:R_0805_2012Metric_Pad1.20x1.40mm_HandSolder" V 7480 3300 50  0001 C CNN

Commit message: More tidyups.
Finished messing with DAC.
Changed inner layers to GND, with 3.3V fill on outers.
Changed lines of the file:
@@
 AR Path="/60687F8A/6068202E/60681FF9" Ref="R503"  Part="1"
 AR Path="/60687F8A/600A04B7/60681FF9" Ref="R603"  Part="1"
-F 0 "R603" V 4100 3000 50  0000 C CNN
+F 0 "R403" V 4100 3000 50  0000 C CNN
 F 1 "12k" V 4200 3000 50  0000 C CNN
 F 2 "Resistor_SMD:R_0805_2012Metric_Pad1.20x1.40mm_HandSolder" V 3930 3000 50  0001 C CNN
@@
 AR Path="/60687F8A/6068202E/60681FFB" Ref="R505"  Part="1"
 AR Path="/60687F8A/600A04B7/60681FFB" Ref="R605"  Part="1"
-F 0 "R605" V 5100 3000 50  0000 C CNN
+F 0 "R405" V 5100 3000 50  0000 C CNN
 F 1 "12k" V 5200 3000 50  0000 C CNN
 F 2 "Resistor_SMD:R_0805_2012Metric_Pad1.20x1.40mm_HandSolder" V 4930 3000 50  0001 C CNN
@@
 AR Path="/60687F8A/6068202E/60681FFC" Ref="R507"  Part="1"
 AR Path="/60687F8A/600A04B7/60681FFC" Ref="R607"  Part="1"
-F 0 "R607" V 6100 3000 50  0000 C CNN
+F 0 "R407" V 6100 3000 50  0000 C CNN
 F 1 "12k" V 6200 3000 50  0000 C CNN
 F 2 "Resistor_SMD:R_0805_2012Metric_Pad1.20x1.40mm_HandSolder" V 5930 3000 50  0001 C CNN
@@
 AR Path="/60687F8A/6068202E/60682000" Ref="#PWR0501"  Part="1"
 AR Path="/60687F8A/600A04B7/60682000" Ref="#PWR0601"  Part="1"
-F 0 "#PWR0601" H 3500 3350 50  0001 C CNN
+F 0 "#PWR0401" H 3500 3350 50  0001 C CNN
 F 1 "GND" H 3505 3427 50  0000 C CNN
 F 2 "" H 3500 3600 50  0001 C CNN
@@
 AR Path="/60687F8A/6068202E/60682001" Ref="#PWR0502"  Part="1"
 AR Path="/60687F8A/600A04B7/60682001" Ref="#PWR0602"  Part="1"
-F 0 "#PWR0602" H 7550 3350 50  0001 C CNN
+F 0 "#PWR0402" H 7550 3350 50  0001 C CNN
 F 1 "GND" H 7555 3427 50  0000 C CNN
 F 2 "" H 7550 3600 50  0001 C CNN
@@
 AR Path="/60687F8A/6068202E/60682002" Ref="R502"  Part="1"
 AR Path="/60687F8A/600A04B7/60682002" Ref="R602"  Part="1"
-F 0 "R602" H 3570 3346 50  0000 L CNN
+F 0 "R402" H 3570 3346 50  0000 L CNN
 F 1 "24k" H 3570 3255 50  0000 L CNN
 F 2 "Resistor_SMD:R_0805_2012Metric_Pad1.20x1.40mm_HandSolder" V 3430 3300 50  0001 C CNN
@@
 AR Path="/60687F8A/6068202E/5F5FD329" Ref="R508"  Part="1"
 AR Path="/60687F8A/600A04B7/5F5FD329" Ref="R608"  Part="1"
-F 0 "R608" H 6570 2746 50  0000 L CNN
+F 0 "R408" H 6570 2746 50  0000 L CNN
 F 1 "24k" H 6570 2655 50  0000 L CNN
 F 2 "Resistor_SMD:R_0805_2012Metric_Pad1.20x1.40mm_HandSolder" V 6430 2700 50  0001 C CNN
@@
 AR Path="/60687F8A/6068202E/60682003" Ref="R506"  Part="1"
 AR Path="/60687F8A/600A04B7/60682003" Ref="R606"  Part="1"
-F 0 "R606" H 5570 2746 50  0000 L CNN
+F 0 "R406" H 5570 2746 50  0000 L CNN
 F 1 "24k" H 5570 2655 50  0000 L CNN
 F 2 "Resistor_SMD:R_0805_2012Metric_Pad1.20x1.40mm_HandSolder" V 5430 2700 50  0001 C CNN
@@
 AR Path="/60687F8A/6068202E/60681FFA" Ref="R504"  Part="1"
 AR Path="/60687F8A/600A04B7/60681FFA" Ref="R604"  Part="1"
-F 0 "R604" H 4570 2746 50  0000 L CNN
+F 0 "R404" H 4570 2746 50  0000 L CNN
 F 1 "24k" H 4570 2655 50  0000 L CNN
 F 2 "Resistor_SMD:R_0805_2012Metric_Pad1.20x1.40mm_HandSolder" V 4430 2700 50  0001 C CNN
@@
 AR Path="/60687F8A/6068202E/5F5F4D05" Ref="R501"  Part="1"
 AR Path="/60687F8A/600A04B7/5F5F4D05" Ref="R601"  Part="1"
-F 0 "R601" H 3570 2746 50  0000 L CNN
+F 0 "R401" H 3570 2746 50  0000 L CNN
 F 1 "24k" H 3570 2655 50  0000 L CNN
 F 2 "Resistor_SMD:R_0805_2012Metric_Pad1.20x1.40mm_HandSolder" V 3430 2700 50  0001 C CNN
@@
 AR Path="/60687F8A/6068202E/60681FFD" Ref="R509"  Part="1"
 AR Path="/60687F8A/600A04B7/60681FFD" Ref="R609"  Part="1"
-F 0 "R609" V 7100 3000 50  0000 C CNN
+F 0 "R409" V 7100 3000 50  0000 C CNN
 F 1 "12k" V 7200 3000 50  0000 C CNN
 F 2 "Resistor_SMD:R_0805_2012Metric_Pad1.20x1.40mm_HandSolder" V 6930 3000 50  0001 C CNN
@@
 AR Path="/60687F8A/6068202E/60681FFF" Ref="R510"  Part="1"
 AR Path="/60687F8A/600A04B7/60681FFF" Ref="R610"  Part="1"
-F 0 "R610" H 7620 3346 50  0000 L CNN
+F 0 "R410" H 7620 3346 50  0000 L CNN
 F 1 "5490" H 7620 3255 50  0000 L CNN
 F 2 "Resistor_SMD:R_0805_2012Metric_Pad1.20x1.40mm_HandSolder" V 7480 3300 50  0001 C CNN
