File: Kicad/video12.sch (KiCad schematic (older format))
At the start: 18 parts, among them J401 DE15HD, U401 THS7316, U402 TPD7S019

Commit message: Added expansion header.
Involved rerouting quite a few things.
Also added through-hole switches for power/reset.
Parts:
- renumbered C401 to C301, C402 to C302, C403 to C303, C404 to C304, C405 to C305, C406 to C306, J401 to J301, R401 to R301, R402 to R302, R403 to R303, R404 to R304, R405 to R305, R406 to R306, R407 to R307, R408 to R308, R409 to R309, U401 to U301, U402 to U302

Commit message: More tidyups.
Finished messing with DAC.
Changed inner layers to GND, with 3.3V fill on outers.
Parts:
- U301: symbol Neotron-Common-Hardware:TPF133A -> Neotron-Common-Hardware:TPF133A-swap
Connections:
- net BLUE_ANA: now also U301.1 (CH1_IN); no longer U301.3 (CH3_IN)
- net RED_ANA: now also U301.3 (CH3_IN); no longer U301.1 (CH1_IN)
- net VGA_BLU: now also U302.5 (VIDEO3); no longer U302.3 (VIDEO1)
- net VGA_RED: now also U302.3 (VIDEO1); no longer U302.5 (VIDEO3)
- net at U301.6 (CH3_OUT): now also R304.2; no longer R306.2
- net at U301.8 (CH1_OUT): now also R306.2; no longer R304.2
Changed lines of the file:
@@
 VGA_DDC_SDA
 NoConn ~ 9650 3600
-$Comp
-L Device:R R304
-U 1 1 60682009
-P 5500 3600
-F 0 "R304" V 5400 3500 50  0000 C CNN
-F 1 "75R" V 5400 3850 50  0000 C CNN
-F 2 "Resistor_SMD:R_0805_2012Metric_Pad1.20x1.40mm_HandSolder" V 5430 3600 50  0001 C CNN
-F 3 "~" H 5500 3600 50  0001 C CNN
-F 4 "0" H 5500 3600 50  0001 C CNN "DNP"
-F 5 "RMCF0805FT75R0-ND" H 5500 3600 50  0001 C CNN "Digikey"
-F 6 "RMCF0805FT75R0" H 5500 3600 50  0001 C CNN "MPN"
-F 7 "Stackpole" H 5500 3600 50  0001 C CNN "Manufacturer"
-F 8 "C20638" H 5500 3600 50  0001 C CNN "LCSC Part#"
-F 9 "1%" H 5500 3600 50  0001 C CNN "Tolerance"
-F 10 "~" H 5500 3600 50  0001 C CNN "Voltage"
-	1    5500 3600
-	0    1    1    0
-$EndComp
-$Comp
-L Device:R R305
-U 1 1 6068200A
-P 5500 3800
-F 0 "R305" V 5400 3700 50  0000 C CNN
-F 1 "75R" V 5400 4050 50  0000 C CNN
-F 2 "Resistor_SMD:R_0805_2012Metric_Pad1.20x1.40mm_HandSolder" V 5430 3800 50  0001 C CNN
-F 3 "~" H 5500 3800 50  0001 C CNN
-F 4 "0" H 5500 3800 50  0001 C CNN "DNP"
-F 5 "RMCF0805FT75R0-ND" H 5500 3800 50  0001 C CNN "Digikey"
-F 6 "RMCF0805FT75R0" H 5500 3800 50  0001 C CNN "MPN"
-F 7 "Stackpole" H 5500 3800 50  0001 C CNN "Manufacturer"
-F 8 "C20638" H 5500 3800 50  0001 C CNN "LCSC Part#"
-F 9 "1%" H 5500 3800 50  0001 C CNN "Tolerance"
-F 10 "~" H 5500 3800 50  0001 C CNN "Voltage"
-	1    5500 3800
-	0    1    1    0
-$EndComp
-$Comp
-L Device:R R306
-U 1 1 6068200B
-P 5500 4000
-F 0 "R306" V 5400 3900 50  0000 C CNN
-F 1 "75R" V 5400 4250 50  0000 C CNN
-F 2 "Resistor_SMD:R_0805_2012Metric_Pad1.20x1.40mm_HandSolder" V 5430 4000 50  0001 C CNN
-F 3 "~" H 5500 4000 50  0001 C CNN
-F 4 "0" H 5500 4000 50  0001 C CNN "DNP"
-F 5 "RMCF0805FT75R0-ND" H 5500 4000 50  0001 C CNN "Digikey"
-F 6 "RMCF0805FT75R0" H 5500 4000 50  0001 C CNN "MPN"
-F 7 "Stackpole" H 5500 4000 50  0001 C CNN "Manufacturer"
-F 8 "C20638" H 5500 4000 50  0001 C CNN "LCSC Part#"
-F 9 "1%" H 5500 4000 50  0001 C CNN "Tolerance"
-F 10 "~" H 5500 4000 50  0001 C CNN "Voltage"
-	1    5500 4000
-	0    1    1    0
-$EndComp
 Wire Wire Line
 	5200 3650 5250 3650
 Wire Wire Line
 	5250 3650 5250 3600
-Wire Wire Line
-	5250 3600 5350 3600
-Wire Wire Line
-	5200 3800 5350 3800
-Wire Wire Line
-	5200 3950 5250 3950
-Wire Wire Line
-	5250 3950 5250 4000
-Wire Wire Line
-	5350 4000 5250 4000
 Wire Wire Line
 	8500 3500 9050 3500
@@
 Wire Wire Line
 	8500 3900 8500 4300
-$Comp
-L power:GND #PWR0311
-U 1 1 6068200D
-P 4600 4550
-F 0 "#PWR0311" H 4600 4300 50  0001 C CNN
-F 1 "GND" H 4605 4377 50  0000 C CNN
-F 2 "" H 4600 4550 50  0001 C CNN
-F 3 "" H 4600 4550 50  0001 C CNN
-	1    4600 4550
-	1    0    0    -1
-$EndComp
-Wire Wire Line
-	4600 4150 4600 4550
-Wire Wire Line
-	4600 3350 4600 3450
 $Comp
 L Device:R R301
@@
 	3950 4000 3950 3950
 Wire Wire Line
-	3950 3950 4050 3950
-Wire Wire Line
 	3500 4000 3500 3800
 Wire Wire Line
@@
 $EndComp
 Wire Wire Line
-	5650 3800 6150 3800
-Wire Wire Line
-	5650 4000 6250 4000
-Connection ~ 6050 3600
-Wire Wire Line
 	6150 5000 6350 5000
-Connection ~ 6250 4000
-Wire Wire Line
-	5650 3600 6050 3600
 Wire Wire Line
 	6150 3800 6150 5000
 Connection ~ 6150 3800
-$Comp
-L Neotron-Common-Hardware:TPF133A U301
-U 1 1 5FEAF8C1
-P 4750 3800
-F 0 "U301" H 5050 4100 50  0000 R CNN
-F 1 "THS7316" H 4300 4100 50  0000 C CNN
-F 2 "Package_SO:SOIC-8_3.9x4.9mm_P1.27mm" H 4750 3250 100 0001 C CNN
-F 3 "https://datasheet.lcsc.com/szlcsc/1810181731_3PEAK-TPF133A-SR_C155446.pdf" H 4050 3750 100 0001 C CNN
-F 4 "Texas Instruments" H 4850 4100 50  0001 C CNN "Manufacturer"
-F 5 "0" H 4750 3800 50  0001 C CNN "DNP"
-F 6 "296-26684-1-ND" H 4750 3800 50  0001 C CNN "Digikey"
-F 7 "THS7316DR" H 4750 3800 50  0001 C CNN "MPN"
-F 8 "595-THS7316DR" H 4750 3800 50  0001 C CNN "Mouser"
-F 9 "C155446" H 4750 3800 50  0001 C CNN "LCSC Part#"
-F 10 "~" H 4750 3800 50  0001 C CNN "Tolerance"
-F 11 "~" H 4750 3800 50  0001 C CNN "Voltage"
-	1    4750 3800
-	1    0    0    -1
-$EndComp
 Wire Wire Line
 	9650 3800 11050 3800
@@
 Text Notes 6350 5800 2    50   Italic 0
 ESD Protection
-Text Notes 2800 3350 0    50   Italic 0
-RGB Buffer\n0.7V p-p inputs\n1.4V p-p outputs, into 75 ohm co-ax
-$Comp
-L power:+3V3 #PWR0310
-U 1 1 5FEFFB4D
-P 4600 3350
-F 0 "#PWR0310" H 4600 3200 50  0001 C CNN
-F 1 "+3V3" H 4615 3523 50  0000 C CNN
-F 2 "" H 4600 3350 50  0001 C CNN
-F 3 "" H 4600 3350 50  0001 C CNN
-	1    4600 3350
-	1    0    0    -1
-$EndComp
 Text Notes 1000 6600 0    50   Italic 0
 TPD7S019
@@
 	2300 6950 2300 6900
 Wire Wire Line
-	6250 4000 9050 4000
-Wire Wire Line
 	6150 3800 9050 3800
-Wire Wire Line
-	6050 3600 9050 3600
 $Comp
 L power:GND #PWR0313
@@
 $EndComp
 Wire Wire Line
-	2475 3950 3950 3950
-Connection ~ 3950 3950
-Wire Wire Line
 	2375 3800 3500 3800
 Connection ~ 3050 3650
@@
 	3050 3650 4050 3650
 Connection ~ 3500 3800
+Connection ~ 9600 5250
+Wire Wire Line
+	9600 5250 7650 5250
+Wire Wire Line
+	9600 5250 11050 5250
+Wire Wire Line
+	6350 5100 6050 5100
+Wire Wire Line
+	6350 4900 6250 4900
+Connection ~ 6250 3600
+Wire Wire Line
+	6250 3600 9050 3600
+Wire Wire Line
+	6050 5100 6050 4000
+Connection ~ 6050 4000
+Wire Wire Line
+	5250 3950 5250 4000
+Wire Wire Line
+	5200 3950 5250 3950
+Wire Wire Line
+	5350 4000 5250 4000
+Wire Wire Line
+	5650 4000 6050 4000
+$Comp
+L Device:R R306
+U 1 1 6068200B
+P 5500 4000
+F 0 "R306" V 5400 3900 50  0000 C CNN
+F 1 "75R" V 5400 4250 50  0000 C CNN
+F 2 "Resistor_SMD:R_0805_2012Metric_Pad1.20x1.40mm_HandSolder" V 5430 4000 50  0001 C CNN
+F 3 "~" H 5500 4000 50  0001 C CNN
+F 4 "0" H 5500 4000 50  0001 C CNN "DNP"
+F 5 "RMCF0805FT75R0-ND" H 5500 4000 50  0001 C CNN "Digikey"
+F 6 "RMCF0805FT75R0" H 5500 4000 50  0001 C CNN "MPN"
+F 7 "Stackpole" H 5500 4000 50  0001 C CNN "Manufacturer"
+F 8 "C20638" H 5500 4000 50  0001 C CNN "LCSC Part#"
+F 9 "1%" H 5500 4000 50  0001 C CNN "Tolerance"
+F 10 "~" H 5500 4000 50  0001 C CNN "Voltage"
+	1    5500 4000
+	0    1    1    0
+$EndComp
+Wire Wire Line
+	5200 3800 5350 3800
+Wire Wire Line
+	5650 3800 6150 3800
+$Comp
+L Device:R R305
+U 1 1 6068200A
+P 5500 3800
+F 0 "R305" V 5400 3700 50  0000 C CNN
+F 1 "75R" V 5400 4050 50  0000 C CNN
+F 2 "Resistor_SMD:R_0805_2012Metric_Pad1.20x1.40mm_HandSolder" V 5430 3800 50  0001 C CNN
+F 3 "~" H 5500 3800 50  0001 C CNN
+F 4 "0" H 5500 3800 50  0001 C CNN "DNP"
+F 5 "RMCF0805FT75R0-ND" H 5500 3800 50  0001 C CNN "Digikey"
+F 6 "RMCF0805FT75R0" H 5500 3800 50  0001 C CNN "MPN"
+F 7 "Stackpole" H 5500 3800 50  0001 C CNN "Manufacturer"
+F 8 "C20638" H 5500 3800 50  0001 C CNN "LCSC Part#"
+F 9 "1%" H 5500 3800 50  0001 C CNN "Tolerance"
+F 10 "~" H 5500 3800 50  0001 C CNN "Voltage"
+	1    5500 3800
+	0    1    1    0
+$EndComp
+Wire Wire Line
+	5250 3600 5350 3600
+Wire Wire Line
+	5650 3600 6250 3600
+$Comp
+L Device:R R304
+U 1 1 60682009
+P 5500 3600
+F 0 "R304" V 5400 3500 50  0000 C CNN
+F 1 "75R" V 5400 3850 50  0000 C CNN
+F 2 "Resistor_SMD:R_0805_2012Metric_Pad1.20x1.40mm_HandSolder" V 5430 3600 50  0001 C CNN
+F 3 "~" H 5500 3600 50  0001 C CNN
+F 4 "0" H 5500 3600 50  0001 C CNN "DNP"
+F 5 "RMCF0805FT75R0-ND" H 5500 3600 50  0001 C CNN "Digikey"
+F 6 "RMCF0805FT75R0" H 5500 3600 50  0001 C CNN "MPN"
+F 7 "Stackpole" H 5500 3600 50  0001 C CNN "Manufacturer"
+F 8 "C20638" H 5500 3600 50  0001 C CNN "LCSC Part#"
+F 9 "1%" H 5500 3600 50  0001 C CNN "Tolerance"
+F 10 "~" H 5500 3600 50  0001 C CNN "Voltage"
+	1    5500 3600
+	0    1    1    0
+$EndComp
+Connection ~ 3950 3950
+Wire Wire Line
+	3950 3950 4050 3950
+Wire Wire Line
+	2475 3950 3950 3950
 Wire Wire Line
 	3500 3800 4050 3800
-Connection ~ 9600 5250
-Wire Wire Line
-	9600 5250 7650 5250
-Wire Wire Line
-	9600 5250 11050 5250
-Wire Wire Line
-	6350 5100 6050 5100
-Wire Wire Line
-	6050 3600 6050 5100
-Wire Wire Line
-	6350 4900 6250 4900
-Wire Wire Line
-	6250 4900 6250 4000
+Text Notes 2800 3350 0    50   Italic 0
+RGB Buffer\n0.7V p-p inputs\n1.4V p-p outputs, into 75 ohm co-ax
+Wire Wire Line
+	4600 4150 4600 4550
+$Comp
+L power:GND #PWR0311
+U 1 1 6068200D
+P 4600 4550
+F 0 "#PWR0311" H 4600 4300 50  0001 C CNN
+F 1 "GND" H 4605 4377 50  0000 C CNN
+F 2 "" H 4600 4550 50  0001 C CNN
+F 3 "" H 4600 4550 50  0001 C CNN
+	1    4600 4550
+	1    0    0    -1
+$EndComp
+$Comp
+L power:+3V3 #PWR0310
+U 1 1 5FEFFB4D
+P 4600 3350
+F 0 "#PWR0310" H 4600 3200 50  0001 C CNN
+F 1 "+3V3" H 4615 3523 50  0000 C CNN
+F 2 "" H 4600 3350 50  0001 C CNN
+F 3 "" H 4600 3350 50  0001 C CNN
+	1    4600 3350
+	1    0    0    -1
+$EndComp
+Wire Wire Line
+	4600 3350 4600 3450
+$Comp
+L Neotron-Common-Hardware:TPF133A-swap U301
+U 1 1 5FEAF8C1
+P 4750 3800
+F 0 "U301" H 5050 4100 50  0000 R CNN
+F 1 "THS7316" H 4300 4100 50  0000 C CNN
+F 2 "Package_SO:SOIC-8_3.9x4.9mm_P1.27mm" H 4750 3250 100 0001 C CNN
+F 3 "https://datasheet.lcsc.com/szlcsc/1810181731_3PEAK-TPF133A-SR_C155446.pdf" H 4050 3750 100 0001 C CNN
+F 4 "Texas Instruments" H 4850 4100 50  0001 C CNN "Manufacturer"
+F 5 "0" H 4750 3800 50  0001 C CNN "DNP"
+F 6 "296-26684-1-ND" H 4750 3800 50  0001 C CNN "Digikey"
+F 7 "THS7316DR" H 4750 3800 50  0001 C CNN "MPN"
+F 8 "595-THS7316DR" H 4750 3800 50  0001 C CNN "Mouser"
+F 9 "C155446" H 4750 3800 50  0001 C CNN "LCSC Part#"
+F 10 "~" H 4750 3800 50  0001 C CNN "Tolerance"
+F 11 "~" H 4750 3800 50  0001 C CNN "Voltage"
+	1    4750 3800
+	1    0    0    -1
+$EndComp
+Wire Wire Line
+	6050 4000 9050 4000
+Wire Wire Line
+	6250 3600 6250 4900
 $EndSCHEMATC
