File: Kicad/dac4.kicad_sch (KiCad schematic)
At the start: 10 parts

Commit message: Cleaned up the part numbers.
Parts:
- R401, R402, R404, R406, R408: Digikey RMCF0805FT2K00CT-ND -> (none); JLCPCB Collection (none) -> Basic; MPN RMCF0805FT2K00 -> 0805W8F2001T5E; Manufacturer Stackpole -> Uniroyal
- R403, R405, R407, R409: Digikey RMCF0805FT1K00CT-ND -> (none); JLCPCB Collection (none) -> Basic; MPN RMCF0805FT1K00 -> 0805W8F1001T5E; Manufacturer Stackpole -> Uniroyal
- R410: Digikey RMCF0805FT300RCT-ND -> (none); JLCPCB Collection (none) -> Basic; MPN RMCF0805FT300R -> 0805W8F3000T5E; Manufacturer Stackpole -> Uniroyal
Changed lines of the file:
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@@
       (effects (font (size 1.27 1.27)) hide)
     )
-    (property "Digikey" "RMCF0805FT2K00CT-ND" (id 5) (at 88.9 68.58 0)
-      (effects (font (size 1.27 1.27)) hide)
-    )
-    (property "MPN" "RMCF0805FT2K00" (id 6) (at 88.9 68.58 0)
-      (effects (font (size 1.27 1.27)) hide)
-    )
-    (property "Manufacturer" "Stackpole" (id 7) (at 88.9 68.58 0)
+    (property "Digikey" "~" (id 5) (at 88.9 68.58 0)
+      (effects (font (size 1.27 1.27)) hide)
+    )
+    (property "MPN" "0805W8F2001T5E" (id 6) (at 88.9 68.58 0)
+      (effects (font (size 1.27 1.27)) hide)
+    )
+    (property "Manufacturer" "Uniroyal" (id 7) (at 88.9 68.58 0)
       (effects (font (size 1.27 1.27)) hide)
     )
@@
       (effects (font (size 1.27 1.27)) hide)
     )
+    (property "JLCPCB Collection" "Basic" (id 12) (at 88.9 68.58 0)
+      (effects (font (size 1.27 1.27)) hide)
+    )
     (pin "1")
     (pin "2")
@@
       (effects (font (size 1.27 1.27)) hide)
     )
-    (property "Digikey" "RMCF0805FT2K00CT-ND" (id 5) (at 165.1 68.58 0)
-      (effects (font (size 1.27 1.27)) hide)
-    )
-    (property "MPN" "RMCF0805FT2K00" (id 6) (at 165.1 68.58 0)
-      (effects (font (size 1.27 1.27)) hide)
-    )
-    (property "Manufacturer" "Stackpole" (id 7) (at 165.1 68.58 0)
+    (property "Digikey" "~" (id 5) (at 165.1 68.58 0)
+      (effects (font (size 1.27 1.27)) hide)
+    )
+    (property "MPN" "0805W8F2001T5E" (id 6) (at 165.1 68.58 0)
+      (effects (font (size 1.27 1.27)) hide)
+    )
+    (property "Manufacturer" "Uniroyal" (id 7) (at 165.1 68.58 0)
       (effects (font (size 1.27 1.27)) hide)
     )
@@
     )
     (property "Mouser" "~" (id 11) (at 165.1 68.58 0)
+      (effects (font (size 1.27 1.27)) hide)
+    )
+    (property "JLCPCB Collection" "Basic" (id 12) (at 165.1 68.58 0)
       (effects (font (size 1.27 1.27)) hide)
     )
@@
       (effects (font (size 1.27 1.27)) hide)
     )
-    (property "Digikey" "RMCF0805FT1K00CT-ND" (id 5) (at 101.6 76.2 0)
-      (effects (font (size 1.27 1.27)) hide)
-    )
-    (property "MPN" "RMCF0805FT1K00" (id 6) (at 101.6 76.2 0)
-      (effects (font (size 1.27 1.27)) hide)
-    )
-    (property "Manufacturer" "Stackpole" (id 7) (at 101.6 76.2 0)
+    (property "Digikey" "~" (id 5) (at 101.6 76.2 0)
+      (effects (font (size 1.27 1.27)) hide)
+    )
+    (property "MPN" "0805W8F1001T5E" (id 6) (at 101.6 76.2 0)
+      (effects (font (size 1.27 1.27)) hide)
+    )
+    (property "Manufacturer" "Uniroyal" (id 7) (at 101.6 76.2 0)
       (effects (font (size 1.27 1.27)) hide)
     )
@@
       (effects (font (size 1.27 1.27)) hide)
     )
+    (property "JLCPCB Collection" "Basic" (id 12) (at 101.6 76.2 0)
+      (effects (font (size 1.27 1.27)) hide)
+    )
     (pin "1")
     (pin "2")
@@
       (effects (font (size 1.27 1.27)) hide)
     )
-    (property "Digikey" "RMCF0805FT2K00CT-ND" (id 5) (at 114.3 68.58 0)
-      (effects (font (size 1.27 1.27)) hide)
-    )
-    (property "MPN" "RMCF0805FT2K00" (id 6) (at 114.3 68.58 0)
-      (effects (font (size 1.27 1.27)) hide)
-    )
-    (property "Manufacturer" "Stackpole" (id 7) (at 114.3 68.58 0)
+    (property "Digikey" "~" (id 5) (at 114.3 68.58 0)
+      (effects (font (size 1.27 1.27)) hide)
+    )
+    (property "MPN" "0805W8F2001T5E" (id 6) (at 114.3 68.58 0)
+      (effects (font (size 1.27 1.27)) hide)
+    )
+    (property "Manufacturer" "Uniroyal" (id 7) (at 114.3 68.58 0)
       (effects (font (size 1.27 1.27)) hide)
     )
@@
     )
     (property "Mouser" "~" (id 11) (at 114.3 68.58 0)
+      (effects (font (size 1.27 1.27)) hide)
+    )
+    (property "JLCPCB Collection" "Basic" (id 12) (at 114.3 68.58 0)
       (effects (font (size 1.27 1.27)) hide)
     )
@@
       (effects (font (size 1.27 1.27)) hide)
     )
-    (property "Digikey" "RMCF0805FT1K00CT-ND" (id 5) (at 127 76.2 0)
-      (effects (font (size 1.27 1.27)) hide)
-    )
-    (property "MPN" "RMCF0805FT1K00" (id 6) (at 127 76.2 0)
-      (effects (font (size 1.27 1.27)) hide)
-    )
-    (property "Manufacturer" "Stackpole" (id 7) (at 127 76.2 0)
+    (property "Digikey" "~" (id 5) (at 127 76.2 0)
+      (effects (font (size 1.27 1.27)) hide)
+    )
+    (property "MPN" "0805W8F1001T5E" (id 6) (at 127 76.2 0)
+      (effects (font (size 1.27 1.27)) hide)
+    )
+    (property "Manufacturer" "Uniroyal" (id 7) (at 127 76.2 0)
       (effects (font (size 1.27 1.27)) hide)
     )
@@
     )
     (property "Mouser" "~" (id 11) (at 127 76.2 0)
+      (effects (font (size 1.27 1.27)) hide)
+    )
+    (property "JLCPCB Collection" "Basic" (id 12) (at 127 76.2 0)
       (effects (font (size 1.27 1.27)) hide)
     )
@@
       (effects (font (size 1.27 1.27)) hide)
     )
-    (property "Digikey" "RMCF0805FT1K00CT-ND" (id 5) (at 152.4 76.2 0)
-      (effects (font (size 1.27 1.27)) hide)
-    )
-    (property "MPN" "RMCF0805FT1K00" (id 6) (at 152.4 76.2 0)
-      (effects (font (size 1.27 1.27)) hide)
-    )
-    (property "Manufacturer" "Stackpole" (id 7) (at 152.4 76.2 0)
+    (property "Digikey" "~" (id 5) (at 152.4 76.2 0)
+      (effects (font (size 1.27 1.27)) hide)
+    )
+    (property "MPN" "0805W8F1001T5E" (id 6) (at 152.4 76.2 0)
+      (effects (font (size 1.27 1.27)) hide)
+    )
+    (property "Manufacturer" "Uniroyal" (id 7) (at 152.4 76.2 0)
       (effects (font (size 1.27 1.27)) hide)
     )
@@
     )
     (property "Mouser" "~" (id 11) (at 152.4 76.2 0)
+      (effects (font (size 1.27 1.27)) hide)
+    )
+    (property "JLCPCB Collection" "Basic" (id 12) (at 152.4 76.2 0)
       (effects (font (size 1.27 1.27)) hide)
     )
@@
       (effects (font (size 1.27 1.27)) hide)
     )
-    (property "Digikey" "RMCF0805FT1K00CT-ND" (id 5) (at 177.8 76.2 0)
-      (effects (font (size 1.27 1.27)) hide)
-    )
-    (property "MPN" "RMCF0805FT1K00" (id 6) (at 177.8 76.2 0)
-      (effects (font (size 1.27 1.27)) hide)
-    )
-    (property "Manufacturer" "Stackpole" (id 7) (at 177.8 76.2 0)
+    (property "Digikey" "~" (id 5) (at 177.8 76.2 0)
+      (effects (font (size 1.27 1.27)) hide)
+    )
+    (property "MPN" "0805W8F1001T5E" (id 6) (at 177.8 76.2 0)
+      (effects (font (size 1.27 1.27)) hide)
+    )
+    (property "Manufacturer" "Uniroyal" (id 7) (at 177.8 76.2 0)
       (effects (font (size 1.27 1.27)) hide)
     )
@@
       (effects (font (size 1.27 1.27)) hide)
     )
+    (property "JLCPCB Collection" "Basic" (id 12) (at 177.8 76.2 0)
+      (effects (font (size 1.27 1.27)) hide)
+    )
     (pin "1")
     (pin "2")
@@
       (effects (font (size 1.27 1.27)) hide)
     )
-    (property "Digikey" "RMCF0805FT300RCT-ND" (id 5) (at 191.77 83.82 0)
-      (effects (font (size 1.27 1.27)) hide)
-    )
-    (property "MPN" "RMCF0805FT300R" (id 6) (at 191.77 83.82 0)
-      (effects (font (size 1.27 1.27)) hide)
-    )
-    (property "Manufacturer" "Stackpole" (id 7) (at 191.77 83.82 0)
+    (property "Digikey" "~" (id 5) (at 191.77 83.82 0)
+      (effects (font (size 1.27 1.27)) hide)
+    )
+    (property "MPN" "0805W8F3000T5E" (id 6) (at 191.77 83.82 0)
+      (effects (font (size 1.27 1.27)) hide)
+    )
+    (property "Manufacturer" "Uniroyal" (id 7) (at 191.77 83.82 0)
       (effects (font (size 1.27 1.27)) hide)
     )
@@
     )
     (property "Mouser" "~" (id 11) (at 191.77 83.82 0)
+      (effects (font (size 1.27 1.27)) hide)
+    )
+    (property "JLCPCB Collection" "Basic" (id 12) (at 191.77 83.82 0)
       (effects (font (size 1.27 1.27)) hide)
     )
@@
       (effects (font (size 1.27 1.27)) hide)
     )
-    (property "Digikey" "RMCF0805FT2K00CT-ND" (id 5) (at 88.9 83.82 0)
-      (effects (font (size 1.27 1.27)) hide)
-    )
-    (property "MPN" "RMCF0805FT2K00" (id 6) (at 88.9 83.82 0)
-      (effects (font (size 1.27 1.27)) hide)
-    )
-    (property "Manufacturer" "Stackpole" (id 7) (at 88.9 83.82 0)
+    (property "Digikey" "~" (id 5) (at 88.9 83.82 0)
+      (effects (font (size 1.27 1.27)) hide)
+    )
+    (property "MPN" "0805W8F2001T5E" (id 6) (at 88.9 83.82 0)
+      (effects (font (size 1.27 1.27)) hide)
+    )
+    (property "Manufacturer" "Uniroyal" (id 7) (at 88.9 83.82 0)
       (effects (font (size 1.27 1.27)) hide)
     )
@@
       (effects (font (size 1.27 1.27)) hide)
     )
+    (property "JLCPCB Collection" "Basic" (id 12) (at 88.9 83.82 0)
+      (effects (font (size 1.27 1.27)) hide)
+    )
     (pin "1")
     (pin "2")
@@
       (effects (font (size 1.27 1.27)) hide)
     )
-    (property "Digikey" "RMCF0805FT2K00CT-ND" (id 5) (at 139.7 68.58 0)
-      (effects (font (size 1.27 1.27)) hide)
-    )
-    (property "MPN" "RMCF0805FT2K00" (id 6) (at 139.7 68.58 0)
-      (effects (font (size 1.27 1.27)) hide)
-    )
-    (property "Manufacturer" "Stackpole" (id 7) (at 139.7 68.58 0)
+    (property "Digikey" "~" (id 5) (at 139.7 68.58 0)
+      (effects (font (size 1.27 1.27)) hide)
+    )
+    (property "MPN" "0805W8F2001T5E" (id 6) (at 139.7 68.58 0)
+      (effects (font (size 1.27 1.27)) hide)
+    )
+    (property "Manufacturer" "Uniroyal" (id 7) (at 139.7 68.58 0)
       (effects (font (size 1.27 1.27)) hide)
     )
@@
       (effects (font (size 1.27 1.27)) hide)
     )
+    (property "JLCPCB Collection" "Basic" (id 12) (at 139.7 68.58 0)
+      (effects (font (size 1.27 1.27)) hide)
+    )

Commit message: Reworked audio circuit.
Based on TLV320AIC23B evaluation board. Removed Pi filters. Used SMD
electrolytic caps for headphone out.
Parts:
- renumbered R404 to R402, R406 to R403, R408 to R404, R403 to R405, R405 to R406, R409 to R408, R402 to R409
Changed lines of the file:
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@@
   (symbol (lib_id "Device:R") (at 165.1 68.58 0) (unit 1)
     (in_bom yes) (on_board yes)
-    (property "Reference" "R408" (id 0) (at 166.878 67.4116 0)
+    (property "Reference" "R404" (id 0) (at 166.878 67.4116 0)
       (effects (font (size 1.27 1.27)) (justify left))
     )
@@
   (symbol (lib_id "Device:R") (at 101.6 76.2 270) (unit 1)
     (in_bom yes) (on_board yes)
-    (property "Reference" "R403" (id 0) (at 101.6 78.74 90))
+    (property "Reference" "R405" (id 0) (at 101.6 78.74 90))
     (property "Value" "1k" (id 1) (at 101.6 81.28 90))
     (property "Footprint" "Resistor_SMD:R_0805_2012Metric_Pad1.20x1.40mm_HandSolder" (id 2) (at 101.6 74.422 90)
@@
   (symbol (lib_id "Device:R") (at 114.3 68.58 0) (unit 1)
     (in_bom yes) (on_board yes)
-    (property "Reference" "R404" (id 0) (at 116.078 67.4116 0)
+    (property "Reference" "R402" (id 0) (at 116.078 67.4116 0)
       (effects (font (size 1.27 1.27)) (justify left))
     )
@@
   (symbol (lib_id "Device:R") (at 127 76.2 270) (unit 1)
     (in_bom yes) (on_board yes)
-    (property "Reference" "R405" (id 0) (at 127 78.74 90))
+    (property "Reference" "R406" (id 0) (at 127 78.74 90))
     (property "Value" "1k" (id 1) (at 127 81.28 90))
     (property "Footprint" "Resistor_SMD:R_0805_2012Metric_Pad1.20x1.40mm_HandSolder" (id 2) (at 127 74.422 90)
@@
   (symbol (lib_id "Device:R") (at 177.8 76.2 270) (unit 1)
     (in_bom yes) (on_board yes)
-    (property "Reference" "R409" (id 0) (at 177.8 78.74 90))
+    (property "Reference" "R408" (id 0) (at 177.8 78.74 90))
     (property "Value" "1k" (id 1) (at 177.8 81.28 90))
     (property "Footprint" "Resistor_SMD:R_0805_2012Metric_Pad1.20x1.40mm_HandSolder" (id 2) (at 177.8 74.422 90)
@@
   (symbol (lib_id "Device:R") (at 88.9 83.82 0) (unit 1)
     (in_bom yes) (on_board yes)
-    (property "Reference" "R402" (id 0) (at 90.678 82.6516 0)
+    (property "Reference" "R409" (id 0) (at 90.678 82.6516 0)
       (effects (font (size 1.27 1.27)) (justify left))
     )
@@
   (symbol (lib_id "Device:R") (at 139.7 68.58 0) (unit 1)
     (in_bom yes) (on_board yes)
-    (property "Reference" "R406" (id 0) (at 141.478 67.4116 0)
-      (effects (font (size 1.27 1.27)) (justify left))
-    )
+    (property "Reference" "R403" (id 0) (at 141.478 67.4116 0)
+      (effects (font (size 1.27 1.27)) (justify left))
+    )

Commit message: Added source resistors on SPI bus.
Also renumbered pages.
Parts:
- renumbered R401 to R501, R402 to R502, R403 to R503, R404 to R504, R405 to R505, R406 to R506, R407 to R507, R408 to R508, R409 to R509, R410 to R510
Changed lines of the file:
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@@
   (symbol (lib_id "Device:R") (at 88.9 68.58 0) (unit 1)
     (in_bom yes) (on_board yes)
-    (property "Reference" "R401" (id 0) (at 90.678 67.4116 0)
+    (property "Reference" "R501" (id 0) (at 90.678 67.4116 0)
       (effects (font (size 1.27 1.27)) (justify left))
     )
@@
   (symbol (lib_id "Device:R") (at 165.1 68.58 0) (unit 1)
     (in_bom yes) (on_board yes)
-    (property "Reference" "R404" (id 0) (at 166.878 67.4116 0)
+    (property "Reference" "R504" (id 0) (at 166.878 67.4116 0)
       (effects (font (size 1.27 1.27)) (justify left))
     )
@@
   (symbol (lib_id "Device:R") (at 101.6 76.2 270) (unit 1)
     (in_bom yes) (on_board yes)
-    (property "Reference" "R405" (id 0) (at 101.6 78.74 90))
+    (property "Reference" "R505" (id 0) (at 101.6 78.74 90))
     (property "Value" "1k" (id 1) (at 101.6 81.28 90))
     (property "Footprint" "Resistor_SMD:R_0805_2012Metric_Pad1.20x1.40mm_HandSolder" (id 2) (at 101.6 74.422 90)
@@
   (symbol (lib_id "Device:R") (at 114.3 68.58 0) (unit 1)
     (in_bom yes) (on_board yes)
-    (property "Reference" "R402" (id 0) (at 116.078 67.4116 0)
+    (property "Reference" "R502" (id 0) (at 116.078 67.4116 0)
       (effects (font (size 1.27 1.27)) (justify left))
     )
@@
   (symbol (lib_id "Device:R") (at 127 76.2 270) (unit 1)
     (in_bom yes) (on_board yes)
-    (property "Reference" "R406" (id 0) (at 127 78.74 90))
+    (property "Reference" "R506" (id 0) (at 127 78.74 90))
     (property "Value" "1k" (id 1) (at 127 81.28 90))
     (property "Footprint" "Resistor_SMD:R_0805_2012Metric_Pad1.20x1.40mm_HandSolder" (id 2) (at 127 74.422 90)
@@
   (symbol (lib_id "Device:R") (at 152.4 76.2 270) (unit 1)
     (in_bom yes) (on_board yes)
-    (property "Reference" "R407" (id 0) (at 152.4 78.74 90))
+    (property "Reference" "R507" (id 0) (at 152.4 78.74 90))
     (property "Value" "1k" (id 1) (at 152.4 81.28 90))
     (property "Footprint" "Resistor_SMD:R_0805_2012Metric_Pad1.20x1.40mm_HandSolder" (id 2) (at 152.4 74.422 90)
@@
   (symbol (lib_id "Device:R") (at 177.8 76.2 270) (unit 1)
     (in_bom yes) (on_board yes)
-    (property "Reference" "R408" (id 0) (at 177.8 78.74 90))
+    (property "Reference" "R508" (id 0) (at 177.8 78.74 90))
     (property "Value" "1k" (id 1) (at 177.8 81.28 90))
     (property "Footprint" "Resistor_SMD:R_0805_2012Metric_Pad1.20x1.40mm_HandSolder" (id 2) (at 177.8 74.422 90)
@@
   (symbol (lib_id "Device:R") (at 191.77 83.82 0) (unit 1)
     (in_bom yes) (on_board yes)
-    (property "Reference" "R410" (id 0) (at 193.548 82.6516 0)
+    (property "Reference" "R510" (id 0) (at 193.548 82.6516 0)
       (effects (font (size 1.27 1.27)) (justify left))
     )
@@
   (symbol (lib_id "power:GND") (at 88.9 91.44 0) (unit 1)
     (in_bom yes) (on_board yes)
-    (property "Reference" "#PWR0401" (id 0) (at 88.9 97.79 0)
+    (property "Reference" "#PWR0501" (id 0) (at 88.9 97.79 0)
       (effects (font (size 1.27 1.27)) hide)
     )
@@
   (symbol (lib_id "power:GND") (at 191.77 91.44 0) (unit 1)
     (in_bom yes) (on_board yes)
-    (property "Reference" "#PWR0402" (id 0) (at 191.77 97.79 0)
+    (property "Reference" "#PWR0502" (id 0) (at 191.77 97.79 0)
       (effects (font (size 1.27 1.27)) hide)
     )
@@
   (symbol (lib_id "Device:R") (at 88.9 83.82 0) (unit 1)
     (in_bom yes) (on_board yes)
-    (property "Reference" "R409" (id 0) (at 90.678 82.6516 0)
+    (property "Reference" "R509" (id 0) (at 90.678 82.6516 0)
       (effects (font (size 1.27 1.27)) (justify left))
     )
@@
   (symbol (lib_id "Device:R") (at 139.7 68.58 0) (unit 1)
     (in_bom yes) (on_board yes)
-    (property "Reference" "R403" (id 0) (at 141.478 67.4116 0)
-      (effects (font (size 1.27 1.27)) (justify left))
-    )
+    (property "Reference" "R503" (id 0) (at 141.478 67.4116 0)
+      (effects (font (size 1.27 1.27)) (justify left))
+    )
